File: K210-M1W/M1W/M1W.kicad_pcb (KiCad board)
At the start: 2 copper layers, 75.7 x 52.8 mm, 22 parts, among them J1 XT60PW-M, Q1 S8050, U1 LM2596S

Commit message: 修复了拓展板BUG
Routing:
- net RGB5050-G: track 7.99 -> 10.5 mm
- net RGB5050-R: track 28.8 -> 30.2 mm
- net RGB5050-B: track 22.3 -> 23.7 mm
- net IO8_LED: track 17.5 -> 16.5 mm
